File: Mochatoo/io.kicad_sch (KiCad schematic)
At the start: 0 parts

Commit message: Added symbols for X201 LCD, daughterboard, keyboard and touchpad connector
Parts:
- added J1: X201_LCD, symbol Connector_Generic:Conn_02x30_Odd_Even
- added J2: X201_daughterboard, symbol Connector_Generic_MountingPin:Conn_01x40_MountingPin
- added J3: X201_keyboard, symbol Connector_Generic_MountingPin:Conn_02x20_Odd_Even_MountingPin
- added J4: X201_touchpad, symbol Connector_Generic:Conn_02x10_Odd_Even
